File: pcb/fr99.kicad_pcb (KiCad board)
At the start: 2 copper layers, 100 x 79.9 mm, 21 parts, among them M1 SD, P1 CONN_02X18, SW2 RESET, U1 541, U2 541, U3 541, U4 377, U5 62256, U6 8515

Commit message: PCB: added values to silkscreen
Other:
- board text added: "Rev. 1a"
- board text removed: "Rev. 1"
Changed lines of the file:
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@@
       (plotreference false)
       (plotvalue true)
-      (plotinvisibletext false)
+      (plotinvisibletext true)
       (padsonsilk false)
       (subtractmaskfromsilk false)
@@
       (effects (font (size 1 1) (thickness 0.15)))
     )
-    (fp_text value SD (at 2.54 2.54) (layer F.Fab)
+    (fp_text value SD (at 2.54 2.54) (layer F.SilkS)
       (effects (font (size 1 1) (thickness 0.15)))
     )
@@
       (effects (font (size 1 1) (thickness 0.15)))
     )
-    (fp_text value 8515 (at 5.08 0.635 180) (layer F.Fab)
+    (fp_text value 8515 (at 5.08 0.635 180) (layer F.SilkS)
       (effects (font (size 1 1) (thickness 0.15)))
     )
@@
       (effects (font (size 1 1) (thickness 0.15)))
     )
-    (fp_text value 377 (at 3.81 0 180) (layer F.Fab)
+    (fp_text value 377 (at 3.81 0 180) (layer F.SilkS)
       (effects (font (size 1 1) (thickness 0.15)))
     )
@@
       (effects (font (size 1 1) (thickness 0.15)))
     )
-    (fp_text value 541 (at 3.81 0 360) (layer F.Fab)
+    (fp_text value 541 (at 3.81 0 360) (layer F.SilkS)
       (effects (font (size 1 1) (thickness 0.15)))
     )
@@
       (effects (font (size 1 1) (thickness 0.15)))
     )
-    (fp_text value BUSY (at -0.635 6.35 180) (layer F.Fab)
+    (fp_text value BUSY (at -0.635 6.35 180) (layer F.SilkS)
       (effects (font (size 1 1) (thickness 0.15)))
     )
@@
       (effects (font (size 1 1) (thickness 0.15)))
     )
-    (fp_text value RESET (at -8.255 -3.175 180) (layer F.Fab)
+    (fp_text value RESET (at -8.255 -3.175 180) (layer F.SilkS)
       (effects (font (size 1 1) (thickness 0.15)))
     )
@@
       (effects (font (size 1 1) (thickness 0.15)))
     )
-    (fp_text value 541 (at 3.81 1.905 360) (layer F.Fab)
+    (fp_text value 541 (at 3.81 1.905 360) (layer F.SilkS)
       (effects (font (size 1 1) (thickness 0.15)))
     )
@@
       (effects (font (size 1 1) (thickness 0.15)))
     )
-    (fp_text value 541 (at 3.81 0.635 180) (layer F.Fab)
+    (fp_text value 541 (at 3.81 0.635 180) (layer F.SilkS)
       (effects (font (size 1 1) (thickness 0.15)))
     )
@@
       (effects (font (size 1 1) (thickness 0.15)))
     )
-    (fp_text value 62256 (at 4.445 0.635 360) (layer F.Fab)
+    (fp_text value 62256 (at 4.445 0.635 360) (layer F.SilkS)
       (effects (font (size 1 1) (thickness 0.15)))
     )
@@
       (effects (font (size 1 1) (thickness 0.15)))
     )
-    (fp_text value 1nF (at -2.54 0 360) (layer F.Fab)
+    (fp_text value 1nF (at -2.54 0 360) (layer F.SilkS)
       (effects (font (size 1 1) (thickness 0.15)))
     )
@@
       (effects (font (size 1 1) (thickness 0.15)))
     )
-    (fp_text value 68 (at 5.08 0 90) (layer F.Fab)
+    (fp_text value 68 (at 5.08 0 90) (layer F.SilkS)
       (effects (font (size 1 1) (thickness 0.15)))
     )
@@
       (effects (font (size 1 1) (thickness 0.15)))
     )
-    (fp_text value 470 (at 5.08 0 90) (layer F.Fab)
+    (fp_text value 470 (at 5.08 0 90) (layer F.SilkS)
       (effects (font (size 1 1) (thickness 0.15)))
     )
@@
       (effects (font (size 1 1) (thickness 0.15)))
     )
-    (fp_text value 10k (at 5.08 0) (layer F.Fab)
+    (fp_text value 10k (at 5.08 0) (layer F.SilkS)
       (effects (font (size 1 1) (thickness 0.15)))
     )
@@
     (effects (font (size 1.016 1.016) (thickness 0.2032)))
   )
-  (gr_text "Rev. 1" (at 191.135 108.585 90) (layer F.SilkS)
-    (effects (font (size 0.762 0.762) (thickness 0.1524)))
+  (gr_text "Rev. 1a" (at 191.135 109.22 90) (layer F.SilkS)
+    (effects (font (size 0.762 0.762) (thickness 0.1524)) (justify left))
   )
   (gr_text "(c) 2016 R. Benzinger" (at 177.8 96.52) (layer F.SilkS)

Commit message: PCB: fixed bank switch (disk access issue)
Connections:
- P1 pad 32: Net-(C7-Pad1) -> Net-(P1-Pad32)
- R1 pad 1: Net-(R1-Pad1) -> Net-(C7-Pad1)
- R1 pad 2: Net-(C7-Pad1) -> Net-(P1-Pad32)
- U4 pad 11: Net-(R1-Pad1) -> Net-(C7-Pad1)
Routing:
- net Net-(P1-Pad32): track 0.00 -> 59.0 mm, vias 0 -> 1
- net Net-(C7-Pad1): track 64.0 -> 16.0 mm, vias 1 -> 0
- net Net-(R1-Pad1): track 11.5 -> 0.00 mm
Other:
- board text added: "Rev. 2"
- board text removed: "Rev. 1a"
